File: SRC/LilyGO_Esp32_Shield.sch (KiCad schematic (older format))
At the start: 47 parts, among them J1 Conn. Flow4, J2 Conn. Flow3, J3 Conn. Flow2, J4 Conn. Flow1, J5 Conn. Pressure, J6 TEMP1, J7 TEMP2, U1 SN74HC14DR

Commit message: lilly go shield complete
Parts:
- gave numbers to parts that had none: 4
Other:
- note added: "ON/OFF SWITCH pads"
Changed lines of the file:
@@
 Wire Wire Line
 	3475 7175 3475 7050
-Text Notes 3475 6700 0    39   ~ 0
-ON/OFF SWITCH
+Text Notes 3225 6750 0    39   ~ 0
+ON/OFF SWITCH pads
 Wire Wire Line
 	3875 7150 4075 7150
@@
 $EndComp
 $Comp
-L GCL_Modules&Devboards:LilyGO_ESP32_TTGO U?
+L GCL_Modules&Devboards:LilyGO_ESP32_TTGO U2
 U 1 1 61971A82
 P 7450 1675
-F 0 "U?" H 7450 2056 50  0000 C CNN
+F 0 "U2" H 7450 2056 50  0000 C CNN
 F 1 "LilyGO_ESP32_TTGO" H 7450 1965 50  0000 C CNN
 F 2 "greencharge-footprints:LILLYGO_ESP32_TTGO" H 6500 1175 50  0001 C CNN
@@
 NoConn ~ 8350 1975
 $Comp
-L dk_Test-Points:RCT-0C TP?
+L dk_Test-Points:RCT-0C TP5
 U 1 1 61A05A6B
 P 3575 7050
-F 0 "TP?" V 3450 7100 50  0000 L CNN
+F 0 "TP5" V 3450 7100 50  0000 L CNN
 F 1 "RCT-0C" V 3500 7075 50  0000 L CNN
 F 2 "digikey-footprints:PROBE_PAD_1206" H 3775 7250 60  0001 L CNN
@@
 $EndComp
 $Comp
-L dk_Test-Points:RCT-0C TP?
+L dk_Test-Points:RCT-0C TP7
 U 1 1 61A1D60E
 P 3775 7150
-F 0 "TP?" V 3700 7125 50  0000 L CNN
+F 0 "TP7" V 3700 7125 50  0000 L CNN
 F 1 "RCT-0C" V 3650 7050 50  0000 L CNN
 F 2 "digikey-footprints:PROBE_PAD_1206" H 3975 7350 60  0001 L CNN
@@
 $EndComp
 $Comp
-L dk_Test-Points:RCT-0C TP?
+L dk_Test-Points:RCT-0C TP6
 U 1 1 61A156F3
 P 3775 6950
-F 0 "TP?" V 3925 6925 50  0000 L CNN
+F 0 "TP6" V 3925 6925 50  0000 L CNN
 F 1 "RCT-0C" V 3850 6850 50  0000 L CNN
 F 2 "digikey-footprints:PROBE_PAD_1206" H 3975 7150 60  0001 L CNN
